File: MiniSumoRC/Boards/MiniSumoMotors.sch (EAGLE design)
At the start: 4 parts, among them U1 ESP32-DEVKIT-V1, U2 ROB-14450, X1 22-23-2021

Commit message: Board
Parts:
- removed U$1: STEP-UP, Boards:STEP-UP
- added M1: MICROMOTOR_N20_L, Boards:MICROMOTOR_N20_L
- added M2: MICROMOTOR_N20_R, Boards:MICROMOTOR_N20_R
- added U3: STEP-UP, Boards:STEP-UP
- added U4: MINI560, Boards:MINI560
Connections:
- removed net N$15: U$1.V_IN, X1-2.S
- new net BAT: U3.V_IN, U4.IN+, X1-2.S
- new net N$12: U3.GND_OUT
- net 3V3: now also U4.OUT+
- net GND: now also U3.GND_IN, U4.IN-, U4.OUT-; no longer U$1.GND_IN, U$1.GND_OUT
- net VM: now also U3.V_OUT; no longer U$1.V_OUT
